File: bistab.kicad_pcb (KiCad board)
At the start: 2 copper layers, 0 parts

Commit message: add component placement
Parts:
- added D1: LED, LED_SMD:LED_0805_2012Metric, F.Cu at (163.4, 62.6)
- added D2: LED, LED_SMD:LED_0805_2012Metric, F.Cu at (165.6, 62.6)
- added J1: Conn_01x02, Connector_PinHeader_2.54mm:PinHeader_1x02_P2.54mm_Vertical, F.Cu at (163.0, 58.2)
- added Q1: NPN, Package_TO_SOT_SMD:SOT-23-3, F.Cu at (160.2, 69.8)
- added Q2: NPN, Package_TO_SOT_SMD:SOT-23-3, F.Cu at (156.8, 73.2)
- added Q3: NPN, Package_TO_SOT_SMD:SOT-23-3, F.Cu at (164.6, 72.4)
- added Q4: NPN, Package_TO_SOT_SMD:SOT-23-3, F.Cu at (168.8, 72.4)
- added R1: 1k, Resistor_SMD:R_0805_2012Metric, F.Cu at (153.6, 71.0)
- added R10: 1k, Resistor_SMD:R_0805_2012Metric, F.Cu at (169.2, 69.6)
- added R2: 1k, Resistor_SMD:R_0805_2012Metric, F.Cu at (163.4, 66.6)
- added R3: 1k, Resistor_SMD:R_0805_2012Metric, F.Cu at (153.0, 73.8)
- added R4: 1k, Resistor_SMD:R_0805_2012Metric, F.Cu at (156.4, 70.4)
- added R5: 1k, Resistor_SMD:R_0805_2012Metric, F.Cu at (160.8, 72.6)
- added R6: 1k, Resistor_SMD:R_0805_2012Metric, F.Cu at (172.0, 70.4)
- added R7: 1k, Resistor_SMD:R_0805_2012Metric, F.Cu at (172.0, 73.8)
- added R8: 1k, Resistor_SMD:R_0805_2012Metric, F.Cu at (165.6, 66.6)
- added R9: 1k, Resistor_SMD:R_0805_2012Metric, F.Cu at (164.6, 69.6)
- added S1: ~, ELO2:PTS645SM43SMTR92 LFS, F.Cu at (156.0, 64.0)
- added S2: ~, ELO2:PTS645SM43SMTR92 LFS, F.Cu at (173.0, 64.2)
Other:
- board outline added: 29 x 24 mm
