File: bistab.kicad_pcb (KiCad board)
At the start: 2 copper layers, 29 x 24 mm, 19 parts, among them J1 Conn_01x02, Q1 NPN, Q2 NPN, Q3 NPN, Q4 NPN

Commit message: add layout
Parts:
- turned R9 to 180 degrees
Routing:
- net VCC: track 0.00 -> 49.0 mm
- net Net-(R1-Pad1): track 0.00 -> 12.5 mm
- net Net-(R6-Pad1): track 0.00 -> 11.0 mm
- net Net-(Q1-B): track 0.00 -> 8.40 mm, vias 0 -> 2
- net Net-(Q1-C): track 0.00 -> 8.13 mm
- net Net-(Q2-E): track 0.00 -> 6.77 mm
- net Net-(Q3-C): track 0.00 -> 5.75 mm
- net Net-(Q4-C): track 0.00 -> 4.43 mm
- net Net-(Q2-B): track 0.00 -> 3.91 mm
- net Net-(Q4-B): track 0.00 -> 3.69 mm
- net Net-(D2-K): track 0.00 -> 2.15 mm
- net Net-(D1-K): track 0.00 -> 2.15 mm
- net Net-(Q2-C): track 0.00 -> 1.92 mm
- net GND: vias 0 -> 39
- added copper zone on B.Cu, net GND
- added copper zone on F.Cu, net GND
